File: SimpleLedProject.kicad_sch (KiCad schematic)
At the start: 4 parts, among them SW1 SW_DPST_x2

Commit message: commit2
Other:
- note added: "Lore ipsum"
- note removed: "bunu yazan tosun okuyana kosun"
Changed lines of the file:
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@@
     (effects (font (size 1.27 1.27)) (justify left bottom))
   )
-  (text "bunu yazan tosun okuyana kosun\n" (at 144.78 135.89 0)
+  (text "Lore ipsum" (at 165.1 135.89 0)
     (effects (font (size 1.27 1.27)) (justify left bottom))
   )
